File: M5StampS3 Breakout/M5StampS3 Breakout.kicad_pcb (KiCad board)
At the start: 2 copper layers, 31.9 x 31.8 mm, 19 parts, among them J1 Conn_01x02, J2 Qwiic_RA, J3 Qwiic_RA, J4 Conn_01x03, J5 Conn_01x04, J6 Conn_01x04, J7 Conn_01x04, U4 XC6220B331MR

Commit message: small update
Parts:
- U1: value ~ -> M5StampS3
Changed lines of the file:
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@@
 		(at 153.08 112.5 180)
 		(property "Reference" "J4"
-			(at -1.27 -1.397 360)
+			(at -1.27 -1.397 0)
 			(layer "F.Fab")
 			(effects
@@
 		)
 		(property "Value" "Conn_01x03"
-			(at -1.27 2.032 360)
+			(at -1.27 2.032 0)
 			(layer "F.Fab")
 			(effects
@@
 		)
 		(property "Footprint" "SparkFun-Connector:1X03"
-			(at 0 0 360)
+			(at 0 0 0)
 			(layer "F.Fab")
 			(hide yes)
@@
 		)
 		(property "Datasheet" ""
-			(at 0 0 360)
+			(at 0 0 0)
 			(layer "F.Fab")
 			(hide yes)
@@
 		)
 		(property "Description" "Generic connector, single row, 01x03, script generated (kicad-library-utils/schlib/autogen/connector/)"
-			(at 0 0 360)
+			(at 0 0 0)
 			(layer "F.Fab")
 			(hide yes)
@@
 			)
 		)
-		(property "Value" "~"
-			(at 3.748203 2.053789 90)
+		(property "Value" "M5StampS3"
+			(at -4 -12.5 180)
 			(unlocked yes)
 			(layer "F.SilkS")
@@
 			)
 		)
-		(sheetname "Root")
-		(sheetfile "M5StampS3 Breakout.kicad_sch")
 		(attr smd)
 		(fp_poly
@@
 			(solder_mask_margin 0.1016)
 		)
-		(model "C:/Users/joel/Desktop/PCB Files/PCB Libraries/M5_Hardware-master/M5_Hardware-master/KiCAD/M5KiCad/M5KiCad.3d/M5STAMP-S3.step"
-			(offset
-				(xyz 0 0 10.6)
-			)
-			(scale
-				(xyz 1 1 1)
-			)
-			(rotate
-				(xyz 0 0 0)
-			)
-		)
 		(model "${KICAD6_3DMODEL_DIR}/Connector_PinSocket_2.54mm.3dshapes/PinSocket_1x09_P2.54mm_Vertical.step"
 			(offset
@@
 		(model "${KICAD6_3DMODEL_DIR}/Connector_PinHeader_2.54mm.3dshapes/PinHeader_1x09_P2.54mm_Vertical.step"
 			(offset
-				(xyz -7 -10 9.5)
+				(xyz -7.5 -10 9.5)
 			)
 			(scale
@@
 			)
 		)
+		(model "C:/Users/joel2/OneDrive/Desktop/Github/PCB_Libraries/Personal_PCB_Libraries/M5_Hardware-master/KiCAD/M5KiCad/M5KiCad.3d/M5STAMP-S3.step"
+			(offset
+				(xyz 0 0 10.5)
+			)
+			(scale
+				(xyz 1 1 1)
+			)
+			(rotate
+				(xyz 0 0 0)
+			)
+		)
 	)
 	(footprint "SparkFun-Hardware:STAND-OFF"
@@
 		)
 		(property "Value" "10UF"
-			(at 0 1.85 360)
+			(at 0 1.85 0)
 			(layer "F.Fab")
 			(effects
@@
 		)
 		(fp_text user "${REFERENCE}"
-			(at 0 0 360)
+			(at 0 0 0)
 			(layer "F.Fab")
 			(effects
@@
 		(tags "resistor")
 		(property "Reference" "R1"
-			(at 0 1.43 360)
+			(at 0 1.43 0)
 			(layer "B.Fab")
 			(effects
@@
 		)
 		(property "Value" "4.7k"
-			(at 0 -1.43 360)
+			(at 0 -1.43 0)
 			(layer "B.Fab")
 			(effects
@@
 		)
 		(property "Footprint" "SparkFun-Resistor:R_0603_1608Metric"
-			(at 0 0 360)
+			(at 0 0 0)
 			(layer "B.Fab")
 			(hide yes)
@@
 		)
 		(property "Datasheet" ""
-			(at 0 0 360)
+			(at 0 0 0)
 			(layer "B.Fab")
 			(hide yes)
@@
 		)
 		(property "Description" "Resistor"
-			(at 0 0 360)
+			(at 0 0 0)
 			(layer "B.Fab")
 			(hide yes)
@@
 		(tags "resistor")
 		(property "Reference" "R2"
-			(at 0 1.43 360)
+			(at 0 1.43 0)
 			(layer "B.Fab")
 			(effects
@@
 		)
 		(property "Value" "4.7k"
-			(at 0 -1.43 360)
+			(at 0 -1.43 0)
 			(layer "B.Fab")
 			(effects
@@
 		)
 		(property "Footprint" "SparkFun-Resistor:R_0603_1608Metric"
-			(at 0 0 360)
+			(at 0 0 0)
 			(layer "B.Fab")
 			(hide yes)
@@
 		)
 		(property "Datasheet" ""
-			(at 0 0 360)
+			(at 0 0 0)
 			(layer "B.Fab")
 			(hide yes)
@@
 		)
 		(property "Description" "Resistor"
-			(at 0 0 360)
+			(at 0 0 0)
 			(layer "B.Fab")
 			(hide yes)
@@
 	)
 	(gr_line
-		(start 166.709 108.75)
-		(end 166.709 111.58)
+		(start 166.709 86.18)
+		(end 166.709 108.75)
 		(stroke
 			(width 0.05)
@@
 	)
 	(gr_line
-		(start 166.709 86.18)
-		(end 166.709 108.75)
+		(start 166.709 108.75)
+		(end 166.709 111.58)
 		(stroke
 			(width 0.05)
